File: hardware/SSS_Motherboard/SSS_Motherboard.kicad_pcb (KiCad board)
At the start: 2 copper layers, 241.3 x 127 mm, 69 parts, among them J1 Screw_Terminal_01x05, J2 Conn_02x06_Odd_Even, J3 Screw_Terminal_01x04, T2 Transformer_2P_3S, U1 STM32G431RBT6, U3 Optocoupler, U4 TPS62933DRLR, U5 TPS54202DDCR, U6 LM675, U7 Optocoupler, U8 TPS62933DRLR, U9 LM675, Y1 X322524MSB4SI

Commit message: manufacturing batch
Parts:
- removed D2, D3, D4: MB6S-50MIL, Diode_SMD:Diode_Bridge_Diotec_ABS
- removed J3: Screw_Terminal_01x04, Project_Lib:4_Connector_11.13_Pitch
- removed JP1, JP2: SolderJumper_2_Open, Jumper:SolderJumper-2_P1.3mm_Open_Pad1.0x1.5mm
- removed U9: LM675, Package_TO_SOT_THT:TO-220-5_P3.4x3.7mm_StaggerOdd_Lead3.8mm_Vertical
- added C33: 100nF, Capacitor_SMD:C_0805_2012Metric, F.Cu at (196.9, 98.3)
- added C34: 100nF, Capacitor_SMD:C_0805_2012Metric, F.Cu at (197.2, 119.8)
- added C35: 220nF, Capacitor_SMD:C_0805_2012Metric, F.Cu at (223.8, 102.3)
- added C36: 100nF, Capacitor_SMD:C_0805_2012Metric, F.Cu at (219.9, 92.3)
- added C37: 220nF, Capacitor_SMD:C_0805_2012Metric, F.Cu at (223.9, 124.3)
- added C38: 100nF, Capacitor_SMD:C_0805_2012Metric, F.Cu at (220.0, 115.3)
- added C39: 100nF, Capacitor_SMD:C_0805_2012Metric, F.Cu at (224.5, 145.3)
- added C40: 100nF, Capacitor_SMD:C_0805_2012Metric, F.Cu at (224.5, 149.1)
- added D1: LED NCD0805R1, Diode_SMD:D_0805_2012Metric, F.Cu at (221.2, 69.6)
- added D10: CD-DF4xxS, Project_Lib:CD-DF4xxS(L), F.Cu at (136.2, 117.6)
- added D11: CD-DF4xxS, Project_Lib:CD-DF4xxS(L), F.Cu at (136.2, 81.6)
- added D5: LED NCD0805R1, Diode_SMD:D_0805_2012Metric, F.Cu at (221.2, 65.1)
- added D6: LED_MCU NCD0805R1, Diode_SMD:D_0805_2012Metric, F.Cu at (176.1, 63.9)
- added D7: LED_SCR2 NCD0805R1, Diode_SMD:D_0805_2012Metric, F.Cu at (240.2, 114.1)
- added D8: LED_SCR1 NCD0805R1, Diode_SMD:D_0805_2012Metric, F.Cu at (240.0, 91.8)
- added D9: CD-DF4xxS, Project_Lib:CD-DF4xxS(L), F.Cu at (136.2, 93.8)
- added J4: Screw_Terminal_01x04, Project_Lib:4_Connector_11.13_Pitch, F.Cu at (53.2, 110.4)
- added JP10: SolderJumper_2_Open, Jumper:SolderJumper-2_P1.3mm_Open_Pad1.0x1.5mm, F.Cu at (209.0, 114.7)
- added JP11: SolderJumper_2_Open, Jumper:SolderJumper-2_P1.3mm_Open_Pad1.0x1.5mm, F.Cu at (175.7, 124.1)
- added JP12: SolderJumper_2_Open, Jumper:SolderJumper-2_P1.3mm_Open_Pad1.0x1.5mm, F.Cu at (176.2, 98.3)
- added JP13: SolderJumper_2_Open, Jumper:SolderJumper-2_P1.3mm_Open_Pad1.0x1.5mm, F.Cu at (220.6, 118.6)
- added JP14: SolderJumper_2_Open, Jumper:SolderJumper-2_P1.3mm_Open_Pad1.0x1.5mm, F.Cu at (220.5, 96.6)
- added JP15: SolderJumper_2_Open, Jumper:SolderJumper-2_P1.3mm_Open_Pad1.0x1.5mm, F.Cu at (214.3, 100.8)
- added JP17: SolderJumper_2_Open, Jumper:SolderJumper-2_P1.3mm_Open_Pad1.0x1.5mm, F.Cu at (215.0, 120.8)
- added JP18: SolderJumper_2_Open, Jumper:SolderJumper-2_P1.3mm_Open_Pad1.0x1.5mm, F.Cu at (235.0, 118.8)
- added JP19: SolderJumper_2_Open, Jumper:SolderJumper-2_P1.3mm_Open_Pad1.0x1.5mm, F.Cu at (236.0, 96.3)
- added JP3: SolderJumper_2_Open, Jumper:SolderJumper-2_P1.3mm_Open_Pad1.0x1.5mm, F.Cu at (127.3, 79.5)
- added JP4: SolderJumper_2_Open, Jumper:SolderJumper-2_P1.3mm_Open_Pad1.0x1.5mm, F.Cu at (127.3, 84.6)
- added JP5: SolderJumper_2_Open, Jumper:SolderJumper-2_P1.3mm_Open_Pad1.0x1.5mm, F.Cu at (127.3, 89.7)
- added JP6: SolderJumper_2_Open, Jumper:SolderJumper-2_P1.3mm_Open_Pad1.0x1.5mm, F.Cu at (127.3, 94.8)
- added JP7: SolderJumper_2_Open, Jumper:SolderJumper-2_P1.3mm_Open_Pad1.0x1.5mm, F.Cu at (127.3, 99.8)
- added JP8: SolderJumper_2_Open, Jumper:SolderJumper-2_P1.3mm_Open_Pad1.0x1.5mm, F.Cu at (127.3, 104.9)
- added JP9: SolderJumper_2_Open, Jumper:SolderJumper-2_P1.3mm_Open_Pad1.0x1.5mm, F.Cu at (211.5, 93.3)
- added R23: 866, Resistor_SMD:R_0805_2012Metric, F.Cu at (193.0, 88.4)
- added R24: 866, Resistor_SMD:R_0805_2012Metric, F.Cu at (192.7, 108.3)
- added R25: 10k, Resistor_SMD:R_0805_2012Metric, F.Cu at (227.6, 87.8)
- added R26: 1k, Resistor_SMD:R_0805_2012Metric, F.Cu at (219.9, 88.6)
- added R27: 1, Resistor_SMD:R_0805_2012Metric, F.Cu at (228.5, 102.3)
- added R28: 100, Resistor_SMD:R_0805_2012Metric, F.Cu at (218.1, 133.1)
- added R29: 500, Resistor_SMD:R_0805_2012Metric, F.Cu at (218.1, 136.8)
- added R30: 250, Resistor_SMD:R_0805_2012Metric, F.Cu at (218.1, 140.6)
- added R31: 1k, Resistor_SMD:R_0805_2012Metric, F.Cu at (224.3, 133.1)
- added R32: 1.5k, Resistor_SMD:R_0805_2012Metric, F.Cu at (224.3, 136.8)
- added R33: 2k, Resistor_SMD:R_0805_2012Metric, F.Cu at (224.4, 140.8)
- added R35: 1, Resistor_SMD:R_0805_2012Metric, F.Cu at (228.2, 124.3)
- added R36: 1k, Resistor_SMD:R_0805_2012Metric, F.Cu at (220.1, 111.3)
- added R37: 10k, Resistor_SMD:R_0805_2012Metric, F.Cu at (227.0, 109.6)
- added TP1: TestPoint_Small, TestPoint:TestPoint_Loop_D2.50mm_Drill1.0mm, F.Cu at (183.0, 85.3)
- added TP2: TestPoint_Small, TestPoint:TestPoint_Loop_D2.50mm_Drill1.0mm, F.Cu at (183.0, 93.3)
- added TP3: TestPoint_Small, TestPoint:TestPoint_Loop_D2.50mm_Drill1.0mm, F.Cu at (171.2, 58.3)
- added TP4: TestPoint_Small, TestPoint:TestPoint_Loop_D2.50mm_Drill1.0mm, F.Cu at (183.0, 98.3)
- added TP5: TestPoint_Small, TestPoint:TestPoint_Loop_D2.50mm_Drill1.0mm, F.Cu at (183.0, 124.3)
- added U2: TLP2345, Package_SO:SO-5-6_4.55x3.7mm_P1.27mm, F.Cu at (196.0, 93.5)
- C10, C12, C14, C18, C21, C25, C31, C7, C8, C9: value 100n -> 100nF
- C11: value 4.7u -> 4.7uF
- C13, C15: value 1u -> 1uF
- C16, C17: value 6.8p -> 6.8pF
- C19, C30: value .1u -> 10nF
- C20, C24, C26, C28, C29: value 22u -> 22uF
- C22: value 68p -> 68pF
- C23, C27, C32: value 47u -> 47uF
- L1, L2: value 600R@100MHz -> BLM21AG601SZ1D (600R@100MHz)
- L3: value 10uH,58.6mOhms -> C476261 (10uH,58.6mOhms); footprint Inductor_SMD:L_0805_2012Metric -> Project_Lib:SRN6045
- L4, L5: value 10uH,21mOhms -> C476261 (10uH,21mOhms); footprint Inductor_SMD:L_0805_2012Metric -> Project_Lib:SRN6045
- R11, R15: value 500k -> 100k
- R14, R7: value 53 -> 500
- U3: value Optocoupler -> TLP2345; footprint Package_DIP:DIP-4_W7.62mm -> Package_SO:SO-5-6_4.55x3.7mm_P1.27mm
- U7: value Optocoupler -> LM675; footprint Package_DIP:DIP-4_W7.62mm -> Package_TO_SOT_THT:TO-220-5_P3.4x3.7mm_StaggerOdd_Lead3.8mm_Vertical
- moved R21 87.4 mm to (240.2, 118.0), turned to 90 degrees
- moved R22 84.9 mm to (240.0, 95.5), turned to 90 degrees
- moved C17 74.9 mm to (185.7, 67.1)
- moved C18 74.6 mm to (188.9, 71.1)
- moved U8 71.0 mm to (160.6, 116.9)
- moved C10 67.0 mm to (189.2, 75.6), turned to 90 degrees
- moved C9 62.9 mm to (207.2, 66.3), turned to -90 degrees
- moved U4 61.1 mm to (159.8, 91.7)
- moved C28 60.7 mm to (151.7, 91.5), turned to 90 degrees
- moved C14 57.2 mm to (201.0, 83.6), turned to 180 degrees
- moved R11 53.2 mm to (214.1, 90.1), turned to 180 degrees
- moved C16 52.6 mm to (185.7, 60.6), turned to 180 degrees
- moved C19 52.4 mm to (214.1, 97.3)
- moved U7 48.7 mm to (224.1, 113.7), turned to -90 degrees
- moved C13 46.8 mm to (205.4, 85.3), turned to 180 degrees
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Connections:
- C16 pad 1: Net-(JP1-B) -> Net-(U1-PF0)
- C17 pad 1: Net-(JP2-A) -> Net-(U1-PF1)
- C19 pad 1: Net-(U6-+) -> Net-(JP9-A)
- C25 pad 1: Net-(U4-SW) -> Net-(U4-BST)
- C25 pad 2: Net-(U4-BST) -> Net-(U4-SW)
- C27 pad 1: 12V_SCR1 -> Net-(JP12-A)
- C30 pad 1: Net-(U9-+) -> Net-(JP10-A)
- C32 pad 1: 12V_SCR2 -> Net-(JP11-A)
- J1 pad 1: SCR1_GATE -> SCR2_GATE
- J1 pad 2: SCR1_CATHODE -> SCR2_CATHODE
- J1 pad 4: SCR2_GATE -> SCR1_GATE
- J1 pad 5: SCR2_CATHODE -> SCR1_CATHODE
- L4 pad 1: 12V_SCR1 -> Net-(JP12-A)
- L5 pad 1: 12V_SCR2 -> Net-(JP11-A)
- R11 pad 2: Net-(U6-+) -> Net-(JP9-B)
- R12 pad 1: 12V_SCR1 -> Net-(JP12-A)
- R14 pad 1: Net-(R14-Pad1) -> Net-(U3-VO)
- R14 pad 2: Net-(U9-+) -> Net-(JP10-A)
- R15 pad 2: Net-(U9-+) -> Net-(JP10-B)
- R16 pad 1: 12V_SCR2 -> Net-(JP11-A)
- R7 pad 1: Net-(R7-Pad1) -> Net-(U2-VO)
- R7 pad 2: Net-(U6-+) -> Net-(JP9-A)
- T2 pad 10: 16V+_SCR2 -> Net-(JP8-A)
- T2 pad 5: 16V-_MCU -> Net-(JP3-A)
- T2 pad 6: 16V+_MCU -> Net-(JP4-A)
- T2 pad 7: 16V-_SCR1 -> Net-(JP5-A)
- T2 pad 8: 16V+_SCR1 -> Net-(JP6-A)
- T2 pad 9: 16V-_SCR2 -> Net-(JP7-A)
- U1 pad 5: Net-(JP1-A) -> Net-(U1-PF0)
- U1 pad 6: Net-(JP2-B) -> Net-(U1-PF1)
- U3 pad 1: PWM1 -> Net-(U3-A)
- U3 pad 3: Net-(R7-Pad1) -> GND_MCU
- U3 pad 4: 12V_SCR1 -> SCR2_CATHODE
- U6 pad 1: Net-(U6-+) -> Net-(JP9-B)
- U6 pad 2: SCR1_GATE -> Net-(U6--)
- U6 pad 3: SCR1_CATHODE -> Net-(JP14-B)
- U6 pad 4: SCR1_GATE -> Net-(JP19-B)
- U6 pad 5: 12V_SCR1 -> Net-(JP15-A)
- U7 pad 1: PWM2 -> Net-(JP10-B)
- U7 pad 2: GND_MCU -> Net-(U7--)
- U7 pad 3: Net-(R14-Pad1) -> Net-(JP13-B)
- U7 pad 4: 12V_SCR2 -> Net-(JP18-B)
- Y1 pad 1: Net-(JP1-B) -> Net-(U1-PF0)
- Y1 pad 3: Net-(JP2-A) -> Net-(U1-PF1)
Routing:
- net 3.3V_MCU: track 24.7 -> 222.9 mm, vias 0 -> 7
- net GND_MCU: track 9.63 -> 158.1 mm, vias 0 -> 21
- net SCR1_CATHODE: track 0.00 -> 86.7 mm, vias 0 -> 17
- net SCR2_CATHODE: track 0.00 -> 80.6 mm, vias 0 -> 17
- net Net-(JP16-A): track 0.00 -> 69.1 mm, vias 0 -> 4
- net PC8: track 0.00 -> 66.2 mm, vias 0 -> 1
- net 12V_SCR2: track 0.00 -> 64.2 mm
- net PC9: track 0.00 -> 61.5 mm, vias 0 -> 1
- net PA10: track 0.00 -> 56.4 mm, vias 0 -> 1
- net NRST: track 0.00 -> 56.1 mm, vias 0 -> 1
- net PWM2: track 0.00 -> 52.1 mm, vias 0 -> 2
- net PA11: track 0.00 -> 51.5 mm, vias 0 -> 1
- net 12V_SCR1: track 0.00 -> 46.4 mm
- net PA12: track 0.00 -> 45.8 mm, vias 0 -> 1
- net JTDI: track 0.00 -> 37.6 mm, vias 0 -> 2
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- added copper zone on B.Cu, net GND_MCU
- added copper zone on F.Cu, net Net-(U4-BST)
- added copper zone on F.Cu, net Net-(U4-SW)
- added copper zone on F.Cu, net Net-(U8-BST)
- added copper zone on F.Cu, net Net-(U8-SW)
- added copper zone on B.Cu, net SCR1_CATHODE
- added copper zone on B.Cu, net SCR2_CATHODE
- added copper zone on F.Cu, net VIN_SCR1
- added copper zone on F.Cu, net VIN_SCR2
