File: hardware/SSS_Motherboard/SSS_Motherboard.kicad_sch (KiCad schematic)
At the start: 72 parts, among them J1 Screw_Terminal_01x05, J2 Conn_02x06_Odd_Even, J3 Screw_Terminal_01x04, T2 Transformer_2P_3S, U1 STM32G431RBT6, U3 Optocoupler, U4 TPS62933DRLR, U5 TPS54202DDCR, U6 LM675, U7 Optocoupler, U8 TPS62933DRLR, U9 LM675, Y1 X322524MSB4SI

Commit message: manufacturing batch
Parts:
- removed D2, D3, D4: MB6S-50MIL, Diode_SMD:Diode_Bridge_Diotec_ABS, symbol Diode_Bridge:ABS2
- removed J3: Screw_Terminal_01x04, Project_Lib:4_Connector_11.13_Pitch, symbol Connector:Screw_Terminal_01x04
- removed JP1, JP2: SolderJumper_2_Open, Jumper:SolderJumper-2_P1.3mm_Open_Pad1.0x1.5mm, symbol Jumper:SolderJumper_2_Open
- removed U3, U7: Optocoupler, Package_DIP:DIP-4_W7.62mm, symbol Isolator:SFH617A-1
- removed U9: LM675, Package_TO_SOT_THT:TO-220-5_P3.4x3.7mm_StaggerOdd_Lead3.8mm_Vertical, symbol Amplifier_Operational:LM675
- added C33, C34, C36, C38, C39, C40: 100nF, Capacitor_SMD:C_0805_2012Metric, symbol Device:C
- added C35, C37: 220nF, Capacitor_SMD:C_0805_2012Metric, symbol Device:C
- added D10, D11, D9: CD-DF4xxS, Project_Lib:CD-DF4xxS(L), symbol Project_Lib:CD-DF4xxS
- added J4: Screw_Terminal_01x04, Project_Lib:4_Connector_11.13_Pitch, symbol Connector:Screw_Terminal_01x04
- added JP10, JP11, JP12, JP13, JP14, JP15, JP17, JP18, JP19, JP3, JP4, JP5, JP6, JP7, JP8, JP9: SolderJumper_2_Open, Jumper:SolderJumper-2_P1.3mm_Open_Pad1.0x1.5mm, symbol Jumper:SolderJumper_2_Open
- added R23, R24: 866, Resistor_SMD:R_0805_2012Metric, symbol Device:R_US
- added R25, R37: 10k, Resistor_SMD:R_0805_2012Metric, symbol Device:R_US
- added R26, R31, R36: 1k, Resistor_SMD:R_0805_2012Metric, symbol Device:R_US
- added R27, R35: 1, Resistor_SMD:R_0805_2012Metric, symbol Device:R_US
- added R28: 100, Resistor_SMD:R_0805_2012Metric, symbol Device:R_US
- added R29: 500, Resistor_SMD:R_0805_2012Metric, symbol Device:R_US
- added R30: 250, Resistor_SMD:R_0805_2012Metric, symbol Device:R_US
- added R32: 1.5k, Resistor_SMD:R_0805_2012Metric, symbol Device:R_US
- added R33: 2k, Resistor_SMD:R_0805_2012Metric, symbol Device:R_US
- added TP1, TP2, TP3, TP4, TP5: TestPoint_Small, TestPoint:TestPoint_Loop_D2.50mm_Drill1.0mm, symbol Connector:TestPoint_Small
- added U2, U3: TLP2345, Package_SO:SO-5-6_4.55x3.7mm_P1.27mm, symbol Project_Lib:TLP2345
- added U7: LM675, Package_TO_SOT_THT:TO-220-5_P3.4x3.7mm_StaggerOdd_Lead3.8mm_Vertical, symbol Amplifier_Operational:LM675
- C10, C12, C14, C18, C21, C25, C31, C7, C8, C9: value 100n -> 100nF
- C11: value 4.7u -> 4.7uF
- C13, C15: value 1u -> 1uF
- C16, C17: value 6.8p -> 6.8pF
- C19, C30: value .1u -> 10nF
- C20, C24, C26, C28, C29: value 22u -> 22uF
- C22: value 68p -> 68pF
- C23, C27, C32: value 47u -> 47uF
- D1, D5: value LED -> LED NCD0805R1; footprint (none) -> Diode_SMD:D_0805_2012Metric
- D6: value LED_MCU -> LED_MCU NCD0805R1; footprint (none) -> Diode_SMD:D_0805_2012Metric
- D7: value LED_SCR2 -> LED_SCR2 NCD0805R1; footprint (none) -> Diode_SMD:D_0805_2012Metric
- D8: value LED_SCR1 -> LED_SCR1 NCD0805R1; footprint (none) -> Diode_SMD:D_0805_2012Metric
- L1, L2: value 600R@100MHz -> BLM21AG601SZ1D (600R@100MHz)
- L3: value 10uH,58.6mOhms -> C476261 (10uH,58.6mOhms); footprint Inductor_SMD:L_0805_2012Metric -> Project_Lib:SRN6045
- L4, L5: value 10uH,21mOhms -> C476261 (10uH,21mOhms); footprint Inductor_SMD:L_0805_2012Metric -> Project_Lib:SRN6045
- R11, R15: value 500k -> 100k
- R14, R7: value 53 -> 500
Connections:
- net 12V_SCR1: now also C33.1, JP12.2 (B), JP15.2 (B), TP4.1, U2.6 (VDD); no longer C27.1, L4.1, R12.1, U6.5 (V+)
- net 12V_SCR2: now also C34.1, JP11.2 (B), JP17.2 (B), TP5.1, U3.6 (VDD); no longer C32.1, L5.1, R16.1
- net 16V+_MCU: now also D11.2, JP4.2 (B); no longer T2.6 (SB)
- net 16V+_SCR1: now also D9.2, JP6.2 (B); no longer T2.8 (SD)
- net 16V+_SCR2: now also D10.2, JP8.2 (B); no longer T2.10 (SD)
- net 16V-_MCU: now also D11.3, JP3.2 (B); no longer T2.5 (SA)
- net 16V-_SCR1: now also D9.3, JP5.2 (B); no longer T2.7 (SC)
- net 16V-_SCR2: now also D10.3, JP7.2 (B); no longer T2.9 (SC)
- net 3.3V_MCU: now also TP3.1
- net GND_MCU: now also D11.4 (-), U2.3 (K), U3.3 (K)
- net GND_SCR1: now also J1.5 (Pin_5), C33.2, C35.2, D9.4 (-), JP14.1 (A), U2.4 (GND); no longer J1.2 (Pin_2), U6.3 (V-)
- net GND_SCR2: now also J1.2 (Pin_2), C34.2, C37.2, D10.4 (-), JP13.1 (A), U3.4 (GND); no longer J1.5 (Pin_5)
- net PWM1: now also R23.2, TP1.1
- net PWM2: now also R24.2, TP2.1
- net SCR1_GATE: now also J1.4 (Pin_4), JP19.1 (A); no longer J1.1 (Pin_1), U6.2 (-), U6.4
- net SCR2_GATE: now also J1.1 (Pin_1), JP18.1 (A); no longer J1.4 (Pin_4)
- net T1: now also J4.1 (Pin_4)
- net T2: now also J4.2 (Pin_2)
- net T3: now also J4.3 (Pin_3)
- net T4: now also J4.4 (Pin_1)
- net VIN_MCU: now also D11.1 (+)
- net VIN_SCR1: now also D9.1 (+)
- net VIN_SCR2: now also D10.1 (+)
- net at R7.1: now also U2.5 (VO)
- net at C30.1, R14.2: now also JP10.1 (A); no longer R15.2
- net at R11.2, U6.1 (+): now also JP9.2 (B), R26.2; no longer C19.1, R7.2
- net at U1.5 (PF0): now also C16.1, Y1.1
- net at U1.6 (PF1): now also C17.1, Y1.3
- net at L4.2, U4.5 (SW): now also C25.2; no longer C25.1
- net at U4.6 (BST): now also C25.1; no longer C25.2
- net at R14.1: now also U3.5 (VO)
- new net: JP3.1 (A), T2.5 (SA)
- new net: JP10.2 (B), R15.2, R36.2, U7.1 (+)
- new net: C38.2, R37.2, U7.2 (-)
- new net: JP13.2 (B), U7.3 (V-)
- new net: JP18.2 (B), R35.1, R37.1, U7.4
- new net: JP17.1 (A), U7.5 (V+)
- new net: JP8.1 (A), T2.10 (SD)
- new net: R23.1, U2.1 (A)
- new net: C27.1, JP12.1 (A), L4.1, R12.1
- new net: R24.1, U3.1 (A)
- new net: C37.1, R35.2
- new net: C19.1, JP9.1 (A), R7.2
- new net: JP5.1 (A), T2.7 (SC)
- new net: JP19.2 (B), R25.1, R27.1, U6.4
- new net: C36.2, R25.2, U6.2 (-)
- new net: C36.1, R26.1
- new net: JP4.1 (A), T2.6 (SB)
- new net: C32.1, JP11.1 (A), L5.1, R16.1
- new net: JP14.2 (B), U6.3 (V-)
- new net: C38.1, R36.1
- new net: JP15.1 (A), U6.5 (V+)
- new net: C35.1, R27.2
- new net: JP7.1 (A), T2.9 (SC)
- new net: JP6.1 (A), T2.8 (SD)
Other:
- note added: "2-10mA input"
- note added: "Debugging Testpoints"
- note added: "Extra Resistors"
- moved on the sheet: C19, C25, R11, R7, U6
